File: hackapet_v4.kicad_pcb (KiCad board)
At the start: 2 copper layers, 56.8 x 66.2 mm, 48 parts, among them J1 Conn_01x02_Socket, J4 USB_C_Receptacle_USB2.0_16P, J7 lipo, Q1 AO3401A, SW1 SW_Push, SW2 SW_Push, SW3 SW_Push, SW4 SW_SPDT, U1 XC6206PxxxMR, U2 ESP-PSRAM32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

Commit message: routed!
Parts:
- removed C22, C23: 10u, Capacitor_SMD:C_0805_2012Metric
- removed D13: LED, LED_SMD:LED_0805_2012Metric
- removed D15: MBR0530, Diode_SMD:D_SOD-123
- removed D2, D6, D8: S-LMBR340FT1G, Diode_SMD:D_0805_2012Metric
- removed Q1: AO3401A, Package_TO_SOT_SMD:SOT-23
- removed R39, R44: 1.5k, Resistor_SMD:R_0805_2012Metric
- removed R43: 5.1k, Resistor_SMD:R_0805_2012Metric
- removed U9: TP4056-42-ESOP8, Package_SO:SOIC-8-1EP_3.9x4.9mm_P1.27mm_EP2.41x3.3mm_ThermalVias
- added C6: 1uF, Capacitor_SMD:C_0805_2012Metric, F.Cu at (196.0, 66.8)
- added C7: 4u7, Capacitor_SMD:C_0805_2012Metric, F.Cu at (201.3, 93.2)
- added C8: 4u7, Capacitor_SMD:C_0805_2012Metric, F.Cu at (195.2, 98.4)
- added D1: LED, LED_SMD:LED_0805_2012Metric, F.Cu at (209.2, 71.9)
- added Q2: 2N7002, Package_TO_SOT_SMD:SOT-23, F.Cu at (202.0, 71.7)
- added R11: 1k5, Resistor_SMD:R_0805_2012Metric, F.Cu at (193.2, 95.5)
- added R12: 3k9, Resistor_SMD:R_0805_2012Metric, F.Cu at (199.3, 98.4)
- added R13: 100R, Resistor_SMD:R_0805_2012Metric, F.Cu at (198.9, 69.6)
- added R14: 10k, Resistor_SMD:R_0805_2012Metric, F.Cu at (201.7, 68.9)
- added R15: 100k, Resistor_SMD:R_0805_2012Metric, F.Cu at (200.3, 91.0)
- added R8: 1k5, Resistor_SMD:R_0805_2012Metric, F.Cu at (196.8, 91.1)
- added R9: 10k, Resistor_SMD:R_0805_2012Metric, F.Cu at (201.3, 95.4)
- added U11: SRV05-4, Package_TO_SOT_SMD:SOT-23-6, F.Cu at (189.8, 61.4)
- added U4: BQ24075RGT, Package_DFN_QFN:VQFN-16-1EP_3x3mm_P0.5mm_EP1.6x1.6mm, F.Cu at (197.2, 94.3)
- BOOT1, C9, RESET1: moved to B.Cu
- C3: value 0.1uF -> 4u7
- C5: value 10uF -> 1uF
- moved J1 44.9 mm to (209.2, 91.2)
- moved D7 28.4 mm to (209.0, 95.0), turned to 180 degrees
- moved C3 26.4 mm to (193.2, 93.3), turned to 180 degrees
- moved R6 26.0 mm to (205.3, 95.0)
- moved BREAKOUT_PINS1 24.9 mm to (189.5, 96.6), turned to -90 degrees
- moved BOOT1 8.79 mm to (179.2, 107.2), turned to 0 degrees
- moved RESET1 8.77 mm to (201.7, 107.1), turned to 0 degrees
- moved C9 7.83 mm to (174.2, 106.2)
- moved C1 5.96 mm to (199.7, 66.7), turned to 0 degrees
- moved J7 5.59 mm to (195.5, 64.5)
- moved U1 3.79 mm to (195.7, 69.6)
- moved R1 2.90 mm to (175.6, 64.1)
- moved R2 2.90 mm to (178.5, 64.1)
- moved R3 2.90 mm to (181.5, 64.1)
- moved R5 1.58 mm to (185.9, 61.3)
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Connections:
- C1 pad 1: GND -> VBUS
- C1 pad 2: Net-(D2-K) -> GND
- C3 pad 1: GND -> +5V
- C3 pad 2: Net-(D2-K) -> GND
- C4 pad 1: Net-(D6-A) -> +3V3
- C5 pad 1: Net-(D6-A) -> +3V3
- J4 pad A4: Net-(D2-A) -> VBUS
- J4 pad A9: Net-(D2-A) -> VBUS
- J4 pad B4: Net-(D2-A) -> VBUS
- J4 pad B9: Net-(D2-A) -> VBUS
- J7 pad 1: Net-(J7-Pin_1) -> +BATT
- SW4 pad 1: Net-(J7-Pin_1) -> Net-(SW4-A)
- SW4 pad 2: +BATT -> SYSOFF
- SW4 pad 3: unconnected-(SW4-C-Pad3) -> GND
- U1 pad 2: Net-(D6-A) -> +3V3
- U1 pad 3: VBUS -> +5V
Routing:
- net +3V3: track 3.18 -> 112.5 mm, vias 0 -> 2
- net VBUS: track 0.00 -> 82.3 mm, vias 0 -> 2
- net GND: track 0.00 -> 69.6 mm, vias 0 -> 10
- net +5V: track 0.00 -> 59.7 mm, vias 0 -> 4
- net Net-(U3-EN): track 6.00 -> 48.9 mm, vias 0 -> 1
- net IO38: track 0.00 -> 42.0 mm, vias 0 -> 1
- net PUSH3: track 7.95 -> 49.7 mm
- net SYSOFF: track 0.00 -> 41.7 mm
- net D-: track 0.00 -> 39.4 mm, vias 0 -> 2
- net LED3: track 0.00 -> 38.0 mm, vias 0 -> 2
- net LED2: track 0.00 -> 37.2 mm, vias 0 -> 2
- net +BATT: track 0.00 -> 37.0 mm
- net D+: track 0.00 -> 36.6 mm, vias 0 -> 2
- net LED1: track 0.00 -> 35.3 mm, vias 0 -> 2
- net IO37: track 0.00 -> 35.3 mm, vias 0 -> 1
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Other:
- board text added: "hackapet v4"
- board text removed: "hackapet v3"

Commit message: add stitching vias
Routing:
- net GND: vias 10 -> 95

Commit message: add keepout, thicken 3v3 to .5
Parts:
- moved R7 3.35 mm to (192.6, 69.6), turned to 90 degrees
- moved R3 1.14 mm to (180.8, 63.2), turned to 45 degrees
- moved R1 1.12 mm to (175.1, 63.1), turned to 45 degrees
- moved R2 1.12 mm to (178.0, 63.1), turned to 45 degrees
- moved J4 0.46 mm to (190.0, 53.3)
Connections:
- SW4 pad 4: (no net) -> GND
- SW4 pad 5: (no net) -> GND
- SW4 pad 6: (no net) -> GND
- U3 pad 15: LED1 -> unconnected-(U3-IO11-Pad15)
- U3 pad 16: LED2 -> unconnected-(U3-IO12-Pad16)
- U3 pad 17: LED3 -> unconnected-(U3-IO13-Pad17)
- U3 pad 40: unconnected-(U3-RXD0-Pad40) -> LED1
- U3 pad 41: unconnected-(U3-IO45-Pad41) -> LED2
- U3 pad 44: unconnected-(U3-IO46-Pad44) -> LED3
Routing:
- net GND: track 69.6 -> 100.0 mm, vias 95 -> 108
- net LED3: track 38.0 -> 17.7 mm
- net LED2: track 37.2 -> 22.9 mm
- net +3V3: track 112.5 -> 125.1 mm, vias 2 -> 3
- net LED1: track 35.3 -> 28.9 mm
- net SLK: track 42.5 -> 45.0 mm
- net Net-(U3-EN): track 48.9 -> 49.8 mm
- net Net-(D4-A): track 3.37 -> 2.70 mm
- net Net-(D3-A): track 3.34 -> 2.67 mm
- net Net-(D5-A): track 3.40 -> 2.75 mm
- net VBUS: track 82.3 -> 82.9 mm

Commit message: update
Parts:
- moved R6 1.14 mm to (206.2, 95.7), turned to -90 degrees
Routing:
- net Net-(J1-Pin_2): track 6.03 -> 4.60 mm
- net GND: track 100.0 -> 101.2 mm
- net +3V3: track 125.1 -> 125.8 mm
- net Net-(D7-A): track 1.80 -> 2.48 mm

Commit message: update
Routing:
- net GND: track 101.2 -> 106.3 mm, vias 108 -> 109
- net +3V3: track 125.8 -> 128.1 mm
- net PUSH3: track 49.7 -> 50.7 mm
- net PUSH2: track 40.6 -> 41.6 mm

Commit message: final updates!
Parts:
- added J2: breakout, Connector_PinHeader_2.54mm:PinHeader_1x02_P2.54mm_Vertical_SMD_Pin1Left, B.Cu at (201.3, 61.5)
Routing:
- net +BATT: track 37.1 -> 44.7 mm
- net GND: track 106.3 -> 107.7 mm
